File: Board/MP1802_GOTEK.kicad_pcb (KiCad board)
At the start: 2 copper layers, 99.1 x 63.5 mm, 39 parts, among them J1 Conn_02x25_Top_Bottom, J2 Conn_02x17_Odd_Even, J3 Conn_02x02_Odd_Even, J4 Conn_02x02_Odd_Even, J5 Barrel_Jack_Switch, J6 Conn_01x04_Male, J7 Conn_01x04_Female, J8 Conn_01x03_Male, SW1 SW_SPDT, U1 74LS06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

Commit message: Revision 0.1.5
Parts:
- removed J4: Conn_02x02_Odd_Even, Connector_PinHeader_2.54mm:PinHeader_2x02_P2.54mm_Vertical
- added R12: 1k, Resistor_THT:R_Axial_DIN0207_L6.3mm_D2.5mm_P2.54mm_Vertical, F.Cu at (76.8, 65.4)
- J3: footprint Connector_PinHeader_2.54mm:PinHeader_2x02_P2.54mm_Vertical -> Connector_PinHeader_2.54mm:PinHeader_2x04_P2.54mm_Vertical
- moved J3 1.27 mm to (138.4, 58.4)
Routing:
- net GND: track 414.1 -> 418.3 mm
- net +5V: track 214.8 -> 212.2 mm
- net /~{READY34}: track 67.0 -> 65.7 mm
- net /~{READY6}: track 41.9 -> 43.2 mm
- net /~{RDATA_RAW}: track 51.7 -> 50.6 mm
- net /+5V_IN: track 25.0 -> 25.6 mm
- net /~{HEADLOAD4}: track 32.8 -> 32.2 mm
Other:
- board text added: "Designed by Sasaji 2022-2023"
- board text added: "Rev. 0.1.5"
- board text removed: "Designed by Sasaji 2022"
- board text removed: "Rev. 0.1.2"
