File: Board/MP1802_GOTEK.kicad_sch (KiCad schematic)
At the start: 35 parts, among them J1 Conn_02x25_Top_Bottom, J2 Conn_02x17_Odd_Even, J3 Conn_02x02_Odd_Even, J4 Conn_02x02_Odd_Even, J5 Barrel_Jack_Switch, J6 Conn_01x04_Male, J7 Conn_01x04_Female, J8 Conn_01x03_Male, SW1 SW_SPDT, U1 74LS06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

Commit message: Revision 0.1.5
Parts:
- removed J3, J4: Conn_02x02_Odd_Even, Connector_PinHeader_2.54mm:PinHeader_2x02_P2.54mm_Vertical, symbol Connector_Generic:Conn_02x02_Odd_Even
- added J3: Conn_02x02_Odd_Even, Connector_PinHeader_2.54mm:PinHeader_2x04_P2.54mm_Vertical, symbol Connector_Generic:Conn_02x04_Odd_Even
- added R12: 1k, Resistor_THT:R_Axial_DIN0207_L6.3mm_D2.5mm_P2.54mm_Vertical, symbol Device:R
Connections:
- net +5V: now also R12.1
- net ~{HEADLOAD2}: now also J3.6 (Pin_6)
- net ~{HEADLOAD4}: now also J3.8 (Pin_8)
- net ~{HEADLOAD}: now also J3.5 (Pin_5), J3.7 (Pin_7)
- net ~{RDATA_RAW}: now also R12.2
- net ~{READY34}: now also J3.4 (Pin_4)
- net ~{READY6}: now also J3.2 (Pin_2)
- net ~{READY}: now also J3.1 (Pin_1), J3.3 (Pin_3)
Other:
- moved on the sheet: R3, U1B
